File: RS485_Converter.kicad_pcb (KiCad board)
At the start: 2 copper layers, 97.8 x 39.4 mm, 22 parts, among them J1 USB_B, J3 Conn_01x02_Pin, J4 Screw_Terminal_01x03, U2 FT232RL, U3 MAX485E

Commit message: Fixed FT232RL connection
Parts:
- added C4: 47p, Capacitor_THT:C_Disc_D4.7mm_W2.5mm_P5.00mm, F.Cu at (115.6, 100.4)
- C1: value 0.1uF -> 4.7u; footprint Capacitor_THT:C_Disc_D5.0mm_W2.5mm_P5.00mm -> Capacitor_THT:C_Disc_D4.7mm_W2.5mm_P5.00mm
- C2: value 0.1uF -> 0.1u; footprint Capacitor_THT:C_Disc_D5.0mm_W2.5mm_P5.00mm -> Capacitor_THT:C_Disc_D4.7mm_W2.5mm_P5.00mm
- C3: value 0.1uF -> 47p; footprint Capacitor_THT:C_Disc_D5.0mm_W2.5mm_P5.00mm -> Capacitor_THT:C_Disc_D4.7mm_W2.5mm_P5.00mm
- moved C3 13.7 mm to (120.7, 100.4), turned to -90 degrees
- moved C1 13.3 mm to (116.8, 95.2), turned to 90 degrees
- moved C2 13.1 mm to (121.9, 95.2), turned to 90 degrees
Connections:
- C3 pad 1: /5V -> Net-(J1-D+)
- U2 pad 19: /5V -> unconnected-(U2-~{RESET}-Pad19)
- U2 pad 26: unconnected-(U2-TEST-Pad26) -> /GND
Routing:
- net /GND: track 188.0 -> 23.5 mm
- net /5V: track 117.5 -> 137.4 mm
- net Net-(J1-D-): track 41.2 -> 33.3 mm
- net Net-(U2-3V3OUT): track 20.7 -> 14.2 mm, vias 2 -> 0
- net Net-(J1-D+): track 39.1 -> 36.9 mm
