File: RS485_Converter.kicad_sch (KiCad schematic)
At the start: 18 parts, among them J1 USB_B, J3 Conn_01x02_Pin, J4 Screw_Terminal_01x03, U2 FT232RL, U3 MAX485E

Commit message: Fixed FT232RL connection
Parts:
- removed C1, C2, C3: 0.1uF, Capacitor_THT:C_Disc_D5.0mm_W2.5mm_P5.00mm, symbol Device:C_Polarized
- added C1: 4.7u, Capacitor_THT:C_Disc_D4.7mm_W2.5mm_P5.00mm, symbol Device:C
- added C2: 0.1u, Capacitor_THT:C_Disc_D4.7mm_W2.5mm_P5.00mm, symbol Device:C
- added C3, C4: 47p, Capacitor_THT:C_Disc_D4.7mm_W2.5mm_P5.00mm, symbol Device:C
Connections:
- net 5V: now also C1.1; no longer U2.19 (~{RESET})
- net GND: now also U2.26 (TEST), C1.2, C2.2, C3.2, C4.2
- net at J1.3 (D+), U2.15 (USBD+): now also C3.1
- net at J1.2 (D-), U2.16 (USBD-): now also C4.1
- net at U2.17 (3V3OUT): now also C2.1
- no-connect marks 0 -> 10
Other:
- moved on the sheet: J1
